Commit message: Cleaning up and Using Gazebo Sim

File: src/assistbot_description/urdf/assistbot_manipulator.xacro (robot description, xacro)
@@ -1,110 +1,4 @@
 <?xml version="1.0" encoding="utf-8"?>
-   <robot name="yahboomcar_X3plus">
-    <link name="base_footprint"/>
-    <link name="imu_link"/>
-    <link name="base_link">
-        <inertial>
-            <origin xyz="-0.0304416859098744 4.23384368655101E-05 0.0448234503408059" rpy="0 0 0"/>
-            <mass value="1.0754239466482"/>
-            <inertia
-                    ixx="0.0208831789264125"
-                    ixy="2.4618093127858E-06"
-                    ixz="0.00616019290028669"
-                    iyy="0.0265621377486244"
-                    iyz="-1.10079499865282E-06"
-                    izz="0.0129535610833954"/>
-        </inertial>
-        <visual>
-            <origin xyz="0 0 0" rpy="0 0 0"/>
-            <geometry>
-                <mesh filename="package://assistbot_description/meshes/X3plus/visual/base_link.STL"/>
-            </geometry>
-            <material name="">
-                <color rgba="0 0.7 0 1"/>
-            </material>
-        </visual>
-        <collision>
-            <origin xyz="0 0 0" rpy="0 0 0"/>
-            <geometry>
-                <mesh filename="package://assistbot_description/meshes/X3plus/collision/base_link.STL"/>
-            </geometry>
-        </collision>
-    </link>
-    <joint name="base_joint" type="fixed">
-        <parent link="base_footprint"/>
-        <child link="base_link"/>
-        <origin xyz="0.0 0.0 0.076" rpy="0 0 0"/>
-    </joint>
-    <joint name="base_imu" type="fixed">
-        <parent link="base_link"/>
-        <child link="imu_link"/>
-        <origin xyz="0.001 0.017 0.0322" rpy="0 3.1415 1.5707"/>
-    </joint>
-    <link name="camera_link">
-        <inertial>
-            <origin xyz="-0.00227617338844674 -6.0192031420306E-06 -0.00616567843043764" rpy="0 0 0"/>
-            <mass value="0.224346273348015"/>
-            <inertia
-                    ixx="0.000420259753235012"
-                    ixy="2.65423313072081E-08"
-                    ixz="-9.20335513714662E-06"
-                    iyy="7.89049803518943E-05"
-                    iyz="6.08195761013683E-09"
-                    izz="0.000414416844201259"/>
-        </inertial>
-        <visual>
-            <origin xyz="0 0 0" rpy="0 0 0"/>
-            <geometry>
-                <mesh filename="package://assistbot_description/meshes/sensor/visual/camera_link.STL"/>
-            </geometry>
-            <material name="">
-                <color rgba="0.7 0.7 0.7 1"/>
-            </material>
-        </visual>
-        <collision>
-            <origin xyz="0 0 0" rpy="0 0 0"/>
-            <geometry>
-                <mesh filename="package://assistbot_description/meshes/sensor/collision/camera_link.STL"/>
-            </geometry>
-        </collision>
-    </link>
-    <joint name="astra_joint" type="fixed">
-        <origin xyz="-0.043645 0 0.41955" rpy="0 0 0"/>
-        <parent link="base_link"/>
-        <child link="camera_link"/>
-    </joint>
-    <link name="laser_link">
-        <inertial>
-            <origin xyz="-0.0193193958962378 0.000338302570666659 -0.01482422577972" rpy="0 0 0"/>
-            <mass value="0.0433399617554554"/>
-            <inertia
-                    ixx="2.03361882296905E-05"
-                    ixy="-3.29493708697467E-07"
-                    ixz="-9.00810512916648E-06"
-                    iyy="4.37540022779682E-05"
-                    iyz="-2.16320544253691E-07"
-                    izz="4.81888233320734E-05"/>
-        </inertial>
-        <visual>
-            <origin xyz="0 0 0" rpy="0 0 0"/>
-            <geometry>
-                <mesh filename="package://assistbot_description/meshes/sensor/visual/laser_link.STL"/>
-            </geometry>
-            <material name="">
-                <color rgba="0.7 0.7 0.7 1"/>
-            </material>
-        </visual>
-        <collision>
-            <origin xyz="0 0 0" rpy="0 0 0"/>
-            <geometry>
-                <mesh filename="package://assistbot_description/meshes/sensor/collision/laser_link.STL"/>
-            </geometry>
-        </collision>
-    </link>
-    <joint name="laser_joint" type="fixed">
-        <origin xyz="0.10478 0 0.0471" rpy="0 0 0"/>
-        <parent link="base_link"/>
-        <child link="laser_link"/>
-    </joint>
+<robot name="assistbot" xmlns:xacro="http://ros.org/wiki/xacro">
     <link name="arm_link1">
         <inertial>
